Commit message: fixed joint axis

File: robot/sq2_ccv.urdf (robot description, URDF)
Before this commit: robot sq2_ccv, 21 links, 20 joints
Joints:
- joint front_casters_pitch_joint: axis 1 0 0 -> 0 1 0
- joint front_pitch2shaft_joint: axis 0 1 0 -> 1 0 0

Commit message: fixing urdf

File: robot/sq2_ccv.urdf (robot description, URDF)
Before this commit: robot sq2_ccv, 21 links, 20 joints
Links:
- link back_casters_pitch_link: mass 5 -> 1.0
- link back_pitch2shaft_link: mass 5 -> 1
- link battery_box_link: mass 10 -> 20
- link front_casters_pitch_link: mass 5 -> 1.0
- link front_pitch2shaft_link: mass 5 -> 1
- link upper_body_link: mass 20 -> 1
Joints:
- joint back_left_caster_joint: axis (none) -> 0 1 0; type fixed -> continuous
- joint back_pitch2shaft_joint: axis 1 0 0 -> (none); limit lower=-0.5 upper=0.5 effort=28 velocity=6.28 -> (none); type revolute -> fixed
- joint back_right_caster_joint: axis (none) -> 0 1 0; type fixed -> continuous
- joint front_left_caster_joint: axis (none) -> 0 1 0; type fixed -> continuous
- joint front_pitch2shaft_joint: axis 1 0 0 -> (none); limit lower=-0.5 upper=0.5 effort=28 velocity=6.28 -> (none); type revolute -> fixed
- joint front_right_caster_joint: axis (none) -> 0 1 0; type fixed -> continuous

Commit message: fixing urdf

File: robot/sq2_ccv.urdf (robot description, URDF)
Before this commit: robot sq2_ccv, 21 links, 20 joints
Joints:
- joint back_pitch2shaft_joint: limit (none) -> lower=-0.5 upper=0.5 effort=28 velocity=6.28
- joint front_pitch2shaft_joint: limit (none) -> lower=-0.5 upper=0.5 effort=28 velocity=6.28

Commit message: add caster support

File: robot/sq2_ccv.urdf (robot description, URDF)
Before this commit: robot sq2_ccv, 21 links, 20 joints
Links:
- added link back_left_caster_support_link; collision box size=0.05 0.05 0.01; visual box size=0.05 0.05 0.01
- added link back_right_caster_support_link; collision box size=0.05 0.05 0.01; visual box size=0.05 0.05 0.01
- added link front_left_caster_support_link; collision box size=0.05 0.05 0.01; visual box size=0.05 0.05 0.01
- added link front_right_caster_support_link; collision box size=0.05 0.05 0.01; visual box size=0.05 0.05 0.01
Joints:
- added joint back_left_caster_support_joint: type continuous, parent back_pitch2shaft_link, child back_left_caster_support_link, origin xyz=0.043 0.167 0.0 rpy=0 0 0, axis 0 0 1
- added joint back_right_caster_support_joint: type continuous, parent back_pitch2shaft_link, child back_right_caster_support_link, origin xyz=0.043 -0.167 0.0 rpy=0 0 0, axis 0 0 1
- added joint front_left_caster_support_joint: type continuous, parent front_pitch2shaft_link, child front_left_caster_support_link, origin xyz=0.043 0.167 0.0 rpy=0 0 0, axis 0 0 1
- added joint front_right_caster_support_joint: type continuous, parent front_pitch2shaft_link, child front_right_caster_support_link, origin xyz=0.043 -0.167 0.0 rpy=0 0 0, axis 0 0 1
- joint back_left_caster_joint: origin xyz=0.043 0.167 -0.010 rpy=0 0 0 -> xyz=0 0 -0.010 rpy=0 0 0; parent back_pitch2shaft_link -> back_left_caster_support_link
- joint back_right_caster_joint: origin xyz=0.043 -0.167 -0.010 rpy=0 0 0 -> xyz=0 0 -0.010 rpy=0 0 0; parent back_pitch2shaft_link -> back_right_caster_support_link
- joint front_left_caster_joint: origin xyz=0.043 0.167 -0.010 rpy=0 0 0 -> xyz=0 0 -0.010 rpy=0 0 0; parent front_pitch2shaft_link -> front_left_caster_support_link
- joint front_right_caster_joint: origin xyz=0.043 -0.167 -0.010 rpy=0 0 0 -> xyz=0 0 -0.010 rpy=0 0 0; parent front_pitch2shaft_link -> front_right_caster_support_link

Commit message: add wheel xacro

File: robot/sq2_ccv.urdf (robot description, URDF)
Before this commit: robot sq2_ccv, 25 links, 24 joints
Links:
- removed link back_caster_cover_link
- removed link front_caster_cover_link
- link front_right_caster_link: geometry collision mesh filename=package://sq2_ccv_choreonoid/meshes/caster.stl; visual cylinder length=0.024 radius=0.0635
Joints:
- removed joint back_caster_cover_link_joint
- removed joint front_caster_cover_link_joint
